Commit message: Adding brabo_description

File: src/brabo_description/urdf/brabo.xacro (robot description, xacro)
@@ -15,5 +15,4 @@
   <xacro:property name="M_SCALE" value="0.001 0.001 0.001"/>
   <xacro:property name="M_PI" value="3.14159"/>
-  <xacro:property name="camera_link" value="0.05" /> <!-- Size of square 'camera' box -->
    <xacro:macro name="inertial_matrix" params="mass">
       <inertial>
@@ -26,5 +25,6 @@
 	    <type>transmission_interface/SimpleTransmission</type>
 	    <joint name="${joint_name}">
-	      <hardwareInterface>hardware_interface/PositionJointInterface</hardwareInterface>
+	      <hardwareInterface>PositionJointInterface</hardwareInterface>
+	      <hardwareInterface>JointStateInterface</hardwareInterface>
 	    </joint>
 	    <actuator name="motor1_${joint_name}">
@@ -77,5 +77,4 @@
       </geometry>
       </collision>>
-	<xacro:inertial_matrix mass="1"/>
   </link>
   <gazebo reference="base_link">
@@ -226,31 +225,4 @@
     <material>Gazebo/Black</material>
   </gazebo>
-   <joint name="camera_joint" type="fixed">
-    <axis xyz="0 1 0" />
-    <origin xyz="0 0 0.075" rpy="0 0 0"/>
-    <parent link="link_5"/>
-    <child link="camera_link"/>
-  </joint>
-  <!-- Camera -->
-  <link name="camera_link">
-    <collision>
-      <origin xyz="0 0 0" rpy="0 0 0"/>
-      <geometry>
-    <box size="${camera_link} ${camera_link} ${camera_link}"/>
-      </geometry>
-    </collision>
-    <visual>
-      <origin xyz="0 0 0" rpy="0 0 0"/>
-      <geometry>
-    <box size="${camera_link} ${camera_link} ${camera_link}"/>
-      </geometry>
-      <material name="red"/>
-    </visual>
-    <inertial>
-      <mass value="1e-5" />
-      <origin xyz="0 0 0" rpy="0 0 0"/>
-      <inertia ixx="1e-6" ixy="0" ixz="0" iyy="1e-6" iyz="0" izz="1e-6" />
-    </inertial>
-  </link>
 <!-- ///////////////////////////////////////////////////////////////////////////////////////////////////////////////////// -->
   <!-- Transmissions for ROS Control -->
@@ -272,43 +244,3 @@
     </plugin>
   </gazebo>
-  <!-- camera -->
-  <gazebo reference="camera_link">
-    <sensor type="camera" name="camera1">
-      <update_rate>30.0</update_rate>
-      <camera name="head">
-        <horizontal_fov>1.3962634</horizontal_fov>
-        <image>
-          <width>800</width>
-          <height>800</height>
-          <format>R8G8B8</format>
-        </image>
-        <clip>
-          <near>0.02</near>
-          <far>300</far>
-        </clip>
-        <noise>
-          <type>gaussian</type>
-          <!-- Noise is sampled independently per pixel on each frame.
-               That pixel's noise value is added to each of its color
-               channels, which at that point lie in the range [0,1]. -->
-          <mean>0.0</mean>
-          <stddev>0.007</stddev>
-        </noise>
-      </camera>
-      <plugin name="camera_controller" filename="libgazebo_ros_camera.so">
-        <alwaysOn>true</alwaysOn>
-        <updateRate>0.0</updateRate>
-        <cameraName>rrbot/camera1</cameraName>
-        <imageTopicName>image_raw</imageTopicName>
-        <cameraInfoTopicName>camera_info</cameraInfoTopicName>
-        <frameName>camera_link</frameName>
-        <hackBaseline>0.07</hackBaseline>
-        <distortionK1>0.0</distortionK1>
-        <distortionK2>0.0</distortionK2>
-        <distortionK3>0.0</distortionK3>
-        <distortionT1>0.0</distortionT1>
-        <distortionT2>0.0</distortionT2>
-      </plugin>
-    </sensor>
-  </gazebo>
 </robot>

File: src/brabo_description/urdf/brabo_gripper.xacro (robot description, xacro)
@@ -37,50 +37,50 @@
 -->
 <!-- ///////////////////////////////////////////////////////////////////////////////////////////////////////////////////// -->
-  <joint name="bottom_joint" type="fixed">
+  <joint name="base_joint" type="fixed">
     <origin xyz="0 0 0" rpy="0 0 0" />
-    <parent link="base_link"/>
-    <child link="bottom_link"/>
-  </joint>
+    <parent link="bottom_link"/>
+    <child link="base_link"/>
+  </joint>
+  <link name="base_link">
+    <visual>
+      <origin xyz=" 0 0 -0.04"  rpy="0 0 0"/>
+      <geometry>
+	       <box size="1 1 0.02" />
+      </geometry>
+      <material name="Brown" />
+    </visual>
+    <collision>
+      <origin xyz=" 0 0 -0.04"  rpy="0 0 0"/>
+      <geometry>
+	       <box size="1 1 0.02" />
+      </geometry>
+      </collision>>
+  </link>
+  <gazebo reference="base_link">
+    <material>Gazebo/White</material>
+  </gazebo>
+<!-- ///////////////////////////////////////////////////////////////////////////////////////////////////////////////////// -->
+  <!-- BASE LINK -->
   <link name="bottom_link">
     <visual>
-      <origin xyz=" 0 0 -0.04"  rpy="0 0 0"/>
-      <geometry>
-	       <box size="1 1 0.02" />
-      </geometry>
-      <material name="Brown" />
-    </visual>
-    <collision>
-      <origin xyz=" 0 0 -0.04"  rpy="0 0 0"/>
-      <geometry>
-	       <box size="1 1 0.02" />
+      <origin xyz="0 0 0" rpy="0 0 0" /> <!-- rotate PI/2 -->
+      <geometry>
+	       <mesh filename="package://brabo_description/meshes/visual/base_link.dae" scale="0.001 0.001 0.001"/>
+      </geometry>
+      <material name="Black" />
+    </visual>
+    <collision>
+      <origin xyz="0 0 .025" rpy="0 0 0" /> <!-- rotate PI/2 -->
+      <geometry>
+	       <cylinder radius=".300" length=".04"/>
       </geometry>
       </collision>>
+	<xacro:inertial_matrix mass="1"/>
   </link>
   <gazebo reference="bottom_link">
     <material>Gazebo/White</material>
   </gazebo>
-<!-- ///////////////////////////////////////////////////////////////////////////////////////////////////////////////////// -->
-  <!-- BASE LINK -->
-  <link name="base_link">
-    <visual>
-      <origin xyz="0 0 0" rpy="0 0 0" /> <!-- rotate PI/2 -->
-      <geometry>
-	       <mesh filename="package://brabo_description/meshes/visual/base_link.dae" scale="0.001 0.001 0.001"/>
-      </geometry>
-      <material name="Black" />
-    </visual>
-    <collision>
-      <origin xyz="0 0 .025" rpy="0 0 0" /> <!-- rotate PI/2 -->
-      <geometry>
-	       <cylinder radius=".300" length=".04"/>
-      </geometry>
-      </collision>>
-	<xacro:inertial_matrix mass="1"/>
-  </link>
-  <gazebo reference="base_link">
-    <material>Gazebo/White</material>
-  </gazebo>
   <joint name="link_1_joint" type="revolute">
-    <parent link="base_link"/>
+    <parent link="bottom_link"/>
     <child link="link_1"/>
     <origin xyz="0 0 0" rpy="0 0 0" />
@@ -224,4 +224,61 @@
   <gazebo reference="link_5">
     <material>Gazebo/Black</material>
+  </gazebo>
+  <xacro:include filename="$(find robotiq_description)/urdf/robotiq_85_gripper.urdf.xacro" />
+  <!-- Robotiq Coupler -->
+  <!--  + Height added by the coupler: 8mm -->
+  <!--  + Reference frame: at the middle (4mm) -->
+  <link name="robotiq_coupler">
+    <visual>
+      <geometry>
+        <mesh filename="package://robotiq_description/meshes/robotiq_85_coupler.stl" />
+      </geometry>
+      <material name="flat_black"/>
+    </visual>
+    <collision>
+      <geometry>
+        <mesh filename="package://robotiq_description/meshes/robotiq_85_coupler.stl" />
+      </geometry>
+    </collision>
+    <inertial>
+      <origin xyz="2.073e-05   1.45286e-03  -1.1049e-03" rpy="0 0 0" />
+      <mass value="0.168" />
+      <inertia ixx="6.69695624e-05" ixy="5.21511788e-09" ixz="-2.74383009e-08"
+               iyy="7.85088161e-05" iyz="5.41105193e-07" izz="1.41819717e-04"/>
+    </inertial>
+  </link>
+  <joint name="robotiq_coupler_joint" type="fixed">
+    <origin xyz="0 0 0.06" rpy="0 0 ${-pi/2.0}" />
+    <parent link="link_5"/>
+    <child link="robotiq_coupler"/>
+  </joint>
+  <gazebo reference="robotiq_coupler">
+    <mu1>0.9</mu1>
+    <mu2>0.9</mu2>
+    <material>Gazebo/FlatBlack</material>
+  </gazebo>
+  <!-- Equivalent to the OpenRAVE manipulator denso_robotiq_85_gripper -->
+  <!-- <link name="denso_robotiq_85_gripper" /> -->
+  <!-- <joint name="manipulator_dummy_joint" type="fixed"> -->
+  <!--   <origin xyz="0 0 0.1441" rpy="0 0 0" /> -->
+  <!--   <parent link="robotiq_coupler"/> -->
+  <!--   <child link="denso_robotiq_85_gripper"/> -->
+  <!-- </joint> -->
+  <!-- Attach the robotiq 85 gripper -->
+  <xacro:robotiq_85_gripper prefix="" parent="robotiq_coupler" >
+    <origin xyz="0 0 0.004" rpy="0 ${-pi/2} ${pi}"/>
+  </xacro:robotiq_85_gripper>
+  <!-- Gazebo grasping plugin -->
+  <gazebo>
+    <gripper name="gazebo_gripper">
+      <grasp_check>
+        <attach_steps>2</attach_steps>    <!-- default: 20 -->
+        <detach_steps>2</detach_steps>    <!-- default: 40 -->
+        <min_contact_count>3</min_contact_count>
+      </grasp_check>
+      <gripper_link>robotiq_85_left_finger_tip_link</gripper_link>
+      <gripper_link>robotiq_85_right_finger_tip_link</gripper_link>
+      <palm_link>robotiq_85_base_link</palm_link>
+    </gripper>
   </gazebo>
 <!-- ///////////////////////////////////////////////////////////////////////////////////////////////////////////////////// -->
